File: VIP_metr.kicad_pcb (KiCad board)
At the start: 2 copper layers, 29.5 x 55 mm, 4 parts, among them J1 Conn_01x03_Pin, J2 Conn_01x02_Pin

Commit message: pcb
Parts:
- removed J1: Conn_01x03_Pin, VIP_metr_Library:conn_x3_pitch2.5
- removed J2: Conn_01x02_Pin, VIP_metr_Library:conn_x2_pitch2.5
- added ?: , , F.Cu at (218.9, 93.8)
- added ?: , , F.Cu at (220.6, 96.3)
- added ?: , , F.Cu at (214.4, 70.6)
- added ?: , , B.Cu at (220.6, 96.3)
- added ?: , , B.Cu at (222.4, 96.3)
- added ?: , , B.Cu at (222.3, 95.0)
- added ?: , , B.Cu at (220.6, 93.8)
- added ?: , , B.Cu at (218.9, 95.0)
- added ?: , , B.Cu at (218.9, 93.8)
- added ?: , , B.Cu at (220.6, 95.0)
- added ?: , , B.Cu at (218.9, 96.3)
- added ?: , , F.Cu at (218.8, 96.3)
- added ?: , , B.Cu at (222.3, 93.8)
- added ?: , , F.Cu at (222.3, 96.3)
- added ?: , , F.Cu at (222.3, 95.0)
- added ?: , , F.Cu at (220.6, 95.0)
- added ?: , , F.Cu at (220.6, 93.8)
- added ?: , , F.Cu at (214.4, 94.6)
- added ?: , , F.Cu at (222.3, 93.8)
- added ?: , , F.Cu at (218.8, 95.0)
- added REF**: SolderJumper-array_P1.3mmPad1.0x1.5mm, Bpi_v2_Lib:SolderJumper-array_P1.3mmPad1.0x1.5mm, F.Cu at (211.9, 85.3)
- added REF**: SolderJumper-array_P1.3mmPad1.0x1.5mm, Bpi_v2_Lib:SolderJumper-array_P1.3mmPad1.0x1.5mm, F.Cu at (211.9, 77.4)
- added REF**: SolderJumper-array_P1.3mmPad1.0x1.5mm, Bpi_v2_Lib:SolderJumper-array_P1.3mmPad1.0x1.5mm, F.Cu at (217.5, 85.3)
- added REF**: SolderJumper-array_P1.3mmPad1.0x1.5mm, Bpi_v2_Lib:SolderJumper-array_P1.3mmPad1.0x1.5mm, F.Cu at (217.5, 77.4)
- added REF**: SolderJumper-array_P1.3mmPad1.0x1.5mm, Bpi_v2_Lib:SolderJumper-array_P1.3mmPad1.0x1.5mm, B.Cu at (216.9, 77.5)
- added REF**: SolderJumper-array_P1.3mmPad1.0x1.5mm, Bpi_v2_Lib:SolderJumper-array_P1.3mmPad1.0x1.5mm, B.Cu at (216.9, 85.3)
- added REF**: SolderJumper-array_P1.3mmPad1.0x1.5mm, Bpi_v2_Lib:SolderJumper-array_P1.3mmPad1.0x1.5mm, B.Cu at (211.2, 85.3)
- added REF**: SolderJumper-array_P1.3mmPad1.0x1.5mm, Bpi_v2_Lib:SolderJumper-array_P1.3mmPad1.0x1.5mm, B.Cu at (211.2, 77.5)
- moved D1 79.9 mm to (214.1, 89.0), turned to -90 degrees
- moved D2 72.0 mm to (209.3, 76.6)
Routing:
- net Earth: track 55.3 -> 20.7 mm
- net Net-(D1-IN+): track 29.8 -> 0.00 mm
- net Net-(D1-IN-): track 28.7 -> 0.00 mm
- net Net-(D1-VCC): track 47.1 -> 23.3 mm
- net I2C_SCL: track 31.1 -> 10.0 mm
- net I2C_SDA: track 35.7 -> 14.8 mm
- added copper zone on F.Cu, net Earth
- added copper zone on In1.Cu, net Earth
- added copper zone on In2.Cu, net Earth
Other:
- board size 29.5 x 55 mm -> 20 x 30 mm
- copper layers 2 -> 4
- board text added: "VIP Metr V0.1"
